Commit message: moving the urdf obstacle

File: robot_description/urdf/obstacles/big_box.urdf (robot description, URDF)
Before this commit: robot big_box, 1 links, 0 joints
Links:
- removed link base_link
- added link obstacle, mass 0.6; collision box size=0.001 0.367 0.22; collision box size=0.001 0.367 0.22
